File: PLACA PRINCIPAL/PLACA PRINCIPAL.kicad_pcb (KiCad board)
At the start: 2 copper layers, 71 x 102 mm, 10 parts, among them J1 Conn_01x01_Pin, U3 ACS712xLCTR-05B

Commit message: placa final
Parts:
- added F1: Fuse, Fuse:Fuseholder_TR5_Littelfuse_No560_No460, F.Cu at (68.9, 47.3)
- moved U3 62.4 mm to (67.8, 36.5)
- moved U2 61.0 mm to (123.6, 54.6)
- moved A1 59.5 mm to (50.3, 65.8)
- moved U4 59.5 mm to (54.3, 108.2)
- moved U1 59.5 mm to (65.5, 51.8)
- moved H1 59.5 mm to (21.1, 31.6)
- moved H2 59.5 mm to (84.1, 31.6)
- moved H3 59.5 mm to (84.1, 125.6)
- moved H4 59.5 mm to (21.1, 125.6)
- moved J1 59.5 mm to (64.5, 62.0)
Routing:
- net GND: track 119.6 -> 104.7 mm
- net Net-(A1-3V3): track 0.00 -> 13.7 mm
- net 31: track 28.9 -> 37.2 mm, vias 0 -> 2
- net 3V3: track 121.4 -> 116.0 mm
- net CS: track 13.0 -> 12.1 mm
- net MOSI: track 70.6 -> 71.4 mm
- net RST: track 20.3 -> 21.1 mm
- net SCK: track 77.8 -> 77.1 mm
- added copper zone on F.Cu, net GND
Other:
- board text added: "ECODESAFIO 2025"
