File: DIVISOR DE TENSION/DIVISOR DE TENSION.kicad_pcb (KiCad board)
At the start: 2 copper layers, 44.6 x 16.6 mm, 12 parts, among them J1 Screw_Terminal_01x02, J2 Conn_01x01_Pin

Commit message: FINAL VERSION 2025
Parts:
- removed H2, H3: MountingHole, MountingHole:MountingHole_2.2mm_M2
- removed R1: 3.3 MEGA, Resistor_THT:R_Axial_DIN0204_L3.6mm_D1.6mm_P7.62mm_Horizontal
- removed R2: 10 MEGA, Resistor_THT:R_Axial_DIN0204_L3.6mm_D1.6mm_P7.62mm_Horizontal
- removed R3: 150k, Resistor_THT:R_Axial_DIN0204_L3.6mm_D1.6mm_P7.62mm_Horizontal
- removed R4: 1 MEGA, Resistor_THT:R_Axial_DIN0204_L3.6mm_D1.6mm_P7.62mm_Horizontal
- removed R5, R6: 47k, Resistor_THT:R_Axial_DIN0204_L3.6mm_D1.6mm_P7.62mm_Horizontal
- added RV1: R_Potentiometer_Trim, Potentiometer_THT:Potentiometer_Bourns_3266Y_Vertical, F.Cu at (58.9, 35.5)
- added RV2: R_Potentiometer_Trim, Potentiometer_THT:Potentiometer_Bourns_3266Y_Vertical, F.Cu at (69.9, 35.5)
- J1: value Screw_Terminal_01x02 -> Conn_01x02_Socket; footprint TerminalBlock:TerminalBlock_MaiXu_MX126-5.0-02P_1x02_P5.00mm -> Connector_JST:JST_EH_B2B-EH-A_1x02_P2.50mm_Vertical
- J2: value Conn_01x01_Pin -> Conn_01x02_Socket; footprint Connector_Pin:Pin_D0.7mm_L6.5mm_W1.8mm_FlatFork -> Connector_JST:JST_EH_B2B-EH-A_1x02_P2.50mm_Vertical
- moved H1 138.8 mm to (55.0, 35.5)
- moved J2 129.7 mm to (66.0, 29.9)
- moved J1 104.3 mm to (68.5, 40.9), turned to 180 degrees
- moved H4 98.4 mm to (79.5, 35.5)
Connections:
- H4 pad 1: Net-(J1-Pin_1) -> GND
- J1 pad 1: Net-(J1-Pin_1) -> GND
- J1 pad 2: Net-(J1-Pin_2) -> V_BAT
- J2 pad 1: Net-(J2-Pin_1) -> VOLTAJE
Routing:
- net Net-(J1-Pin_1): track 19.2 -> 0.00 mm
- net VOLTAJE: track 0.00 -> 13.3 mm
- net Net-(J1-Pin_2): track 9.60 -> 0.00 mm
- net Net-(R4-Pad1): track 9.05 -> 0.00 mm
- net Net-(R2-Pad1): track 9.05 -> 0.00 mm
- net V_BAT: track 0.00 -> 7.38 mm
- net Net-(J2-Pin_1): track 7.22 -> 0.00 mm
- net Net-(R1-Pad2): track 5.00 -> 0.00 mm
- net Net-(R1-Pad1): track 3.57 -> 0.00 mm
- added copper zone on B.Cu, net GND
- removed copper zone on B.Cu, net Net-(J1-Pin_1)
Other:
- board size 44.6 x 16.6 mm -> 33.5 x 15.7 mm
